File: control/control.kicad_pcb (KiCad board)
At the start: 4 copper layers, 45.7 x 39.4 mm, 90 parts, among them M1 LMR62014, M2 LM46001, M3 STM32F4XX, M4 TPS736XX, M5 SN65HVD23X, P1 GND/VDD, P2 VOLTAGE, P3 INTERFACE, P4 POWER/FETS, P5 SENSOR_A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

Commit message: Fixed a few small mistakes.
Parts:
- C6: value 100nF -> 10nF
- C8: value 10nF -> 100nF
Changed lines of the file:
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@@
-(kicad_pcb (version 4) (host pcbnew 4.0.2-stable)
+(kicad_pcb (version 4) (host pcbnew 4.0.4-stable)
   (general
     (links 215)
     (no_connects 0)
-    (area 96.4311 52.395 155.955 99.770001)
+    (area 97.079999 60.249999 142.950001 99.770001)
     (thickness 1.6)
     (drawings 6)
@@
       (effects (font (size 0.635 0.635) (thickness 0.127)))
     )
-    (fp_text value 100nF (at 0 -1.397 180) (layer F.SilkS) hide
+    (fp_text value 10nF (at 0 -1.397 180) (layer F.SilkS) hide
       (effects (font (size 0.635 0.635) (thickness 0.127)))
     )
@@
       (effects (font (size 0.635 0.635) (thickness 0.127)))
     )
-    (fp_text value 10nF (at 0 -1.397 270) (layer F.SilkS) hide
+    (fp_text value 100nF (at 0 -1.397 270) (layer F.SilkS) hide
       (effects (font (size 0.635 0.635) (thickness 0.127)))
     )
@@
         (xy 135.89 85.09) (xy 135.89 93.345) (xy 142.24 93.345) (xy 142.24 99.06) (xy 104.14 99.06)
         (xy 104.14 95.25) (xy 106.68 92.71) (xy 129.54 92.71) (xy 130.81 91.44) (xy 130.81 88.9)
-        (xy 128.905 86.995) (xy 128.905 83.058) (xy 133.858 83.058) (xy 135.89 85.09)
+        (xy 128.905 86.995) (xy 128.905 83.058) (xy 133.858 83.058)
       )
     )
@@
         (xy 135.89 85.09) (xy 135.89 93.345) (xy 142.24 93.345) (xy 142.24 99.06) (xy 104.14 99.06)
         (xy 104.14 95.25) (xy 106.68 92.71) (xy 129.54 92.71) (xy 130.81 91.44) (xy 130.81 88.9)
-        (xy 128.905 86.995) (xy 128.905 83.058) (xy 133.858 83.058) (xy 135.89 85.09)
+        (xy 128.905 86.995) (xy 128.905 83.058) (xy 133.858 83.058)
       )
     )

Commit message: Added revison 3.
Parts:
- removed P8: ANALOG, foot:PLS2
- removed PAD1 (x3): VAL**, foot:PAD1
- added C46: 100nF, foot:SM0603, B.Cu at (119.4, 95.9)
- added M6: REF30XX, foot:SOT23, F.Cu at (103.5, 94.6)
- added Q1: BC857C, foot:SOT23, F.Cu at (123.2, 67.3)
- C1, C32, C44, C45, R14, R15, R18, R19, R20, R21: moved to F.Cu
- C12, C7: value 20pF -> 12pF; moved to F.Cu
- C19: value 10uF -> 100nF; footprint foot:SM1210 -> foot:SM0603; moved to F.Cu
- C24: value 100nF -> 4.7uF; footprint foot:SM0603 -> foot:SM0805
- C26, C28: value 47uF -> 100nF; footprint foot:SM1210 -> foot:SM0603
- C40, D2, D3, D4: moved to B.Cu
- C9: value 220pF -> 22pF
- M1: value LMR62014 -> TPS61040
- M4: footprint foot:SOT223 -> foot:SOT23-5
- R3: value 270 -> 470
- R4: value 11K -> 11K 1%
- R5, R6: value 100K -> 100K 1%
- R7: value 27K -> 27K 1%
- Z1: value 8MHz -> 12MHz; footprint foot:HC-49US -> foot:SMD_Z3225
- moved P7 43.2 mm to (99.1, 87.6), turned to 90 degrees
- moved C1 40.4 mm to (137.2, 64.1), turned to 90 degrees
- moved L1 39.5 mm to (133.3, 65.4), turned to 180 degrees
- moved R18 39.3 mm to (101.6, 87.6), turned to 270 degrees
- moved D1 39.2 mm to (128.9, 64.8), turned to 0 degrees
- moved C5 37.3 mm to (135.9, 69.2)
- moved C17 34.7 mm to (128.3, 67.9), turned to 0 degrees
- moved M1 33.2 mm to (133.3, 69.2), turned to 270 degrees
- moved M5 31.5 mm to (106.7, 87.6), turned to 90 degrees
- moved R4 30.3 mm to (130.2, 71.8), turned to 270 degrees
- moved C9 30.0 mm to (128.3, 71.8)
- moved R5 29.7 mm to (126.4, 71.8)
- moved C19 29.2 mm to (122.6, 69.8), turned to 180 degrees
- moved C38 28.3 mm to (109.2, 87.6), turned to 90 degrees
- moved C45 27.0 mm to (135.9, 73.7)
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Connections:
- net ADC_IN0 renamed ADC_E
- net ADC_IN1 renamed ADC_B
- net ADC_IN12 renamed ADC_NTC
- net ADC_IN13 renamed ADC_A
- net ADC_IN2 renamed ADC_U
- net DAC_OUT1 renamed DAC_B
- net DAC_OUT2 renamed DAC_A
- net SWDCLK renamed SWCLK
- C17 pad 1: +12V -> Net-(C17-Pad1)
- C26 pad 1: +5V -> +3.3VREF
- C28 pad 1: +5V -> +3.3VREF
- C6 pad 1: +3.3V -> +3.3VREF
- C8 pad 1: +3.3V -> +3.3VREF
- C9 pad 1: Net-(C9-Pad1) -> +12V
- C9 pad 2: +12V -> Net-(C9-Pad2)
- D1 pad 1: +12V -> Net-(C17-Pad1)
- M1 pad 3: Net-(C9-Pad1) -> Net-(C9-Pad2)
- M1 pad 4: Net-(M1-Pad4) -> 12V_EN
- M2 pad 11: Net-(M2-Pad11) -> (no net)
- M2 pad 6: Net-(M2-Pad6) -> (no net)
- M2 pad 8: Net-(M2-Pad8) -> (no net)
- M3 pad 13: +3.3V -> +3.3VREF
- M3 pad 17: ADC_IN3 -> (no net)
- M3 pad 2: Net-(M3-Pad2) -> (no net)
- M3 pad 22: Net-(M3-Pad22) -> (no net)
- M3 pad 23: Net-(M3-Pad23) -> (no net)
- M3 pad 24: Net-(M3-Pad24) -> (no net)
- M3 pad 25: Net-(M3-Pad25) -> (no net)
- M3 pad 26: Net-(M3-Pad26) -> (no net)
- M3 pad 27: Net-(M3-Pad27) -> (no net)
- M3 pad 28: Net-(M3-Pad28) -> 12V_EN
- M3 pad 29: Net-(M3-Pad29) -> (no net)
- M3 pad 3: Net-(M3-Pad3) -> (no net)
- M3 pad 30: Net-(M3-Pad30) -> (no net)
- M3 pad 33: Net-(M3-Pad33) -> (no net)
- M3 pad 4: Net-(M3-Pad4) -> (no net)
- M3 pad 40: Net-(M3-Pad40) -> (no net)
- M3 pad 44: Net-(M3-Pad44) -> (no net)
- M3 pad 45: Net-(M3-Pad45) -> (no net)
- M3 pad 50: Net-(M3-Pad50) -> (no net)
- M3 pad 53: Net-(M3-Pad53) -> (no net)
- M3 pad 54: Net-(M3-Pad54) -> (no net)
- M3 pad 55: LED_RED -> (no net)
- M3 pad 56: LED_GREEN -> (no net)
- M3 pad 57: LED_BLUE -> LED_R
- M3 pad 58: Net-(M3-Pad58) -> LED_G
- M3 pad 59: Net-(M3-Pad59) -> LED_B
- M3 pad 8: Net-(M3-Pad8) -> (no net)
- M3 pad 9: Net-(M3-Pad9) -> (no net)
- M4 pad 2: +3.3V -> GND
- M4 pad 3: GND -> +5V
- M4 pad 5: +5V -> +3.3V
- P4 pad 1: GND -> +36V
- P4 pad 10: GND -> +12V
- P4 pad 2: +36V -> GND
- P4 pad 3: FET_AH -> FET_AL
- P4 pad 4: FET_AL -> FET_AH
- P4 pad 5: FET_BH -> FET_BL
- P4 pad 6: FET_BL -> FET_BH
- P4 pad 7: FET_CH -> FET_CL
- P4 pad 8: FET_CL -> FET_CH
- P4 pad 9: +12V -> GND
- P5 pad 2: +3.3V -> +3.3VREF
- R1 pad 1: Net-(M1-Pad4) -> +5V
- R1 pad 2: +5V -> Net-(Q1-Pad1)
- R10 pad 1: EN_B -> +3.3V
- R10 pad 2: +3.3V -> EN_C
- R12 pad 1: EN_C -> +3.3V
- R12 pad 2: +3.3V -> EN_B
- R19 pad 1: LED_RED -> LED_R
- R20 pad 1: LED_GREEN -> LED_G
- R21 pad 1: LED_BLUE -> LED_B
- R4 pad 2: Net-(C9-Pad1) -> Net-(C9-Pad2)
- R5 pad 1: +12V -> Net-(C9-Pad2)
- R5 pad 2: Net-(C9-Pad1) -> +12V
- R8 pad 2: Net-(M3-Pad28) -> 12V_EN
- R9 pad 1: EN_A -> +3.3V
- R9 pad 2: +3.3V -> EN_A
- U1 pad 8: +3.3V -> +3.3VREF
Routing:
- net +12V: track 73.1 -> 18.8 mm, vias 7 -> 0
- net GND: track 112.1 -> 61.7 mm, vias 61 -> 34
- net +5V: track 71.3 -> 34.7 mm, vias 5 -> 11
- net +3.3V: track 72.0 -> 51.1 mm, vias 14 -> 12
- net Net-(C44-Pad1): track 8.92 -> 24.0 mm, vias 1 -> 2
- net 12V_EN: track 0.00 -> 14.9 mm, vias 0 -> 1
- net +3.3VREF: track 0.00 -> 14.9 mm, vias 0 -> 3
- net LED_GREEN: track 11.2 -> 0.00 mm, vias 1 -> 0
- net LED_BLUE: track 10.8 -> 0.00 mm, vias 1 -> 0
- net Net-(D4-Pad2): track 13.7 -> 3.43 mm
- net ADC_NTC: track 19.2 -> 9.19 mm
- net Net-(D3-Pad2): track 12.6 -> 3.43 mm
- net Net-(C7-Pad2): track 7.03 -> 15.1 mm
- net Net-(C9-Pad2): track 0.00 -> 7.64 mm
- net HVIN: track 9.60 -> 1.98 mm
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- added copper zone on In2.Cu, net +3.3VREF
- removed copper zone on B.Cu, net +12V
- removed copper zone on F.Cu, net +12V
Other:
- board text added: "PMC rev3"
- board text added: "R3"
