File: power/power.sch (KiCad schematic (older format))
At the start: 70 parts, among them M1 HIP2101, M2 HIP2101, M3 HIP2101, P1 PLS_10, P2 PLS_3, P3 PLS_3, P4 C, P5 A, P6 B, P7 VDD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

Commit message: Added revison 3.
Parts:
- removed C16, C17: 1uF, foot:SM0805, symbol C
- removed R1, R2, R3, R4, R5, R6: 10K, foot:SM0603, symbol R
- C21, C25, C29: value 0.1uF -> 100nF
- M1, M2, M3: value HIP2101 -> UCC27211A; footprint foot:SO8 -> foot:SON8
- R10, R11, R12, R13, R14, R9: value 2 -> 1
Connections:
- net +12V: now also P1.10; no longer P1.9
- net +36V: now also P1.1; no longer P1.2
- net FET_AH: now also P1.4; no longer P1.3
- net FET_AL: now also P1.3; no longer P1.4
- net FET_BH: now also P1.6; no longer P1.5
- net FET_BL: now also P1.5; no longer P1.6
- net FET_CH: now also P1.8; no longer P1.7
- net FET_CL: now also P1.7; no longer P1.8
- net PGND: now also P1.2, P1.9; no longer P1.1, P1.10
Other:
- moved on the sheet: C1, C10, C11, C12, C13, C14, C15, C2, C21, C25, C29, C3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

Commit message: Fixed a little mistake.
Parts:
- C18: Designation (none) -> EEU-FR1J681L; Part Number EEU-FR1J681L -> (none)
- R10, R11, R12, R13, R14, R9: value 1 -> 2
Changed lines of the file:
@@
 F 2 "foot:CE135L" H 12600 1700 60  0001 C CNN
 F 3 "~" H 12600 1700 60  0000 C CNN
-F 4 "EEU-FR1J681L" V 12600 1700 60  0001 C CNN "Part Number"
+F 4 "EEU-FR1J681L" V 12600 1700 60  0001 C CNN "Designation"
 	1    12600 1700
 	0    -1   -1   0
@@
 P 7350 1850
 F 0 "R10" H 7450 1700 60  0000 C CNN
-F 1 "1" H 7250 1700 60  0000 C CNN
+F 1 "2" H 7250 1700 60  0000 C CNN
 F 2 "foot:SM0603" H 7350 1850 60  0001 C CNN
 F 3 "" H 7350 1850 60  0000 C CNN
@@
 P 7350 1650
 F 0 "R9" H 7450 1800 60  0000 C CNN
-F 1 "1" H 7250 1800 60  0000 C CNN
+F 1 "2" H 7250 1800 60  0000 C CNN
 F 2 "foot:SM0603" H 7350 1650 60  0001 C CNN
 F 3 "" H 7350 1650 60  0000 C CNN
@@
 P 7350 5950
 F 0 "R14" H 7450 5800 60  0000 C CNN
-F 1 "1" H 7250 5800 60  0000 C CNN
+F 1 "2" H 7250 5800 60  0000 C CNN
 F 2 "foot:SM0603" H 7350 5950 60  0001 C CNN
 F 3 "" H 7350 5950 60  0000 C CNN
@@
 P 7350 5750
 F 0 "R13" H 7450 5900 60  0000 C CNN
-F 1 "1" H 7250 5900 60  0000 C CNN
+F 1 "2" H 7250 5900 60  0000 C CNN
 F 2 "foot:SM0603" H 7350 5750 60  0001 C CNN
 F 3 "" H 7350 5750 60  0000 C CNN
@@
 P 7350 3850
 F 0 "R12" H 7450 3700 60  0000 C CNN
-F 1 "1" H 7250 3700 60  0000 C CNN
+F 1 "2" H 7250 3700 60  0000 C CNN
 F 2 "foot:SM0603" H 7350 3850 60  0001 C CNN
 F 3 "" H 7350 3850 60  0000 C CNN
@@
 P 7350 3650
 F 0 "R11" H 7450 3800 60  0000 C CNN
-F 1 "1" H 7250 3800 60  0000 C CNN
+F 1 "2" H 7250 3800 60  0000 C CNN
 F 2 "foot:SM0603" H 7350 3650 60  0001 C CNN
 F 3 "" H 7350 3650 60  0000 C CNN
