File: pmc.sch (KiCad schematic (older format))
At the start: 142 parts, among them M1 LM46001, M2 TPS61040, M3 STM32F4XX, M4 REF30XX, M5 TPS736XX, M6 SN65HVD23X, M7 UCC27211A, M8 UCC27211A, M9 UCC27211A, P1 BOOT, P10 CONN4, P11 DEBUG, P2 PWM, P3 HALL, P4 SPI, P5 CAN, P6 CONN4, P7 CONN4, P8 CONN4, P9 CONN4, Q1 BC857C, Q2 IPT007N06N, Q3 IPT007N06N, Q4 IPT007N06N, Q5 IPT007N06N, Q6 IPT007N06N, Q7 IPT007N06N, U1 AD8539, U2 AD8539, U3 AD8417, U4 AD8417

Commit message: Small fixes in schematic and pcb.
Parts:
- removed C29: 100nF 25v, foot:SM0603, symbol C
- added R43, R44: 10K, foot:SM0603, symbol R
- C11: value 100nF 15v -> 100nF 25v
- C32, C33, C34: value 100nF -> 100nF 25v
- C57, C59, C61: value 100nF 100v -> 2.2uF 100v; footprint foot:SM0805 -> foot:SM1206
- M2: PN (none) -> blablah
- M3: value STM32F4XX -> STM32F405RG
- M4: value REF30XX -> REF3033
- M5: value TPS736XX -> TPS73633
- M6: value SN65HVD23X -> SN65HVD233
Connections:
- net +3.3V: now also R43.1, R44.1
- net PWM_INA: now also R43.2
- net PWM_INB: now also R44.2
- net BEMF_A renamed VOLTAGE_A
- net BEMF_B renamed VOLTAGE_B
- net BEMF_C renamed VOLTAGE_C
- net SENSOR_A renamed CURRENT_A
- net SENSOR_B renamed CURRENT_B
- net SENSOR_U renamed VOLTAGE_U
Other:
- note added: "Hardrware specification:\n* PCB dimension 47mm x 45mm\n* Single supply from 5V to 40V\n* Motor current up to 50A\n* PWM frequency 20kHz to 80kHz"
- note added: "Usage: CAN bus only"
- note added: "Usage:\n* Flash STM32 microcontroller\n* Debug via SWD\n* Configure and control via USART\n"
- note added: "Usage:\n* Hall Sensors\n* Quadrature Encoder\n* NTC Resistor (motor temperature)"
- note added: "Usage:\n* RC servo PWM input\n* I2C to any peripheral"
- note added: "Usage:\n* SPI to any peripheral\n* ADC/DAC\n* GPIO (e.g. control buttons)"
- moved on the sheet: C39, C40, C41, C42, C43, C58, C60, M6, P1, P11, P2, P3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

Commit message: Minor fixing.
Connections:
- net PWM_INA renamed I2C_SCL
- net PWM_INB renamed I2C_SDA
Changed lines of the file:
@@
 Sheet 1 1
 Title "Phobia Motor Controller"
-Date "2018-04-01"
+Date "2018-04-03"
 Rev "4"
 Comp "Roman Belov"
@@
 U 1 1 59D9345F
 P 4750 2100
-F 0 "C20" V 4800 2250 60  0000 C CNN
+F 0 "C20" V 4850 2250 60  0000 C CNN
 F 1 "220pF" V 4450 2200 60  0000 C CNN
 F 2 "foot:SM0603" H 4750 2100 60  0001 C CNN
@@
 $EndComp
 Text GLabel 9150 13700 0    60   Input ~ 0
-PWM_INA
+I2C_SCL
 $Comp
 L +5V #PWR061
@@
 	12000 10800 12000 11000
 Text GLabel 8900 9450 2    60   Input ~ 0
-PWM_INA
+I2C_SCL
 $Comp
 L R R40
@@
 $EndComp
 Text GLabel 9000 9750 2    60   Input ~ 0
-PWM_INB
+I2C_SDA
 Wire Wire Line
 	6550 9550 7150 9550
@@
 $EndComp
 Text GLabel 9700 13800 0    60   Input ~ 0
-PWM_INB
+I2C_SDA
 Wire Wire Line
 	10200 13800 9700 13800

Commit message: Fixed SilkS layers again.
Parts:
- C1, C10, C13, C14, C15, C19, C2, C21, C3, C30, C31, C42, C45, C47, C49, C50, C52, C54, R39: footprint foot:SM0805 -> foot:SM-0805
- C11, C12, C16, C17, C20, C22, C23, C24, C25, C27, C32, C33, C34, C35, C36, C37, C38, C39, C4, C40, C41, C43, C44, C46, C48, C5, C51, C53, C55, C6, C64, C65, C66, C7, C8, C9, D2, R1, R10, R11, R12, R13, R14, R15, R16, R17, R18, R19, R2, R20, R21, R22, R23, R24, R25, R26, R27, R28, R29, R3, R30, R31, R32, R33, R34, R38, R4, R40, R41, R42, R43, R44, R5, R6, R7, R8, R9: footprint foot:SM0603 -> foot:SM-0603
- C18, C26, C28: footprint foot:SM1210 -> foot:SM-1210
- C56, C58, C60: footprint foot:CE135L -> foot:CE135-E
- C57, C59, C61, R35: footprint foot:SM1206 -> foot:SM-1206
- L1: footprint foot:COIL3 -> foot:COIL-3
- L2: footprint foot:COIL8 -> foot:COIL-8
- M1: footprint foot:HTSSOP16 -> foot:HTSSOP-16
- M2, M5: footprint foot:SOT23-5 -> foot:SOT-23-5
- M4, Q1: footprint foot:SOT23 -> foot:SOT-23
- M6: footprint foot:SO8 -> foot:SO-8
- M7, M8, M9: footprint foot:SON8 -> foot:SON-8
- P1, P2: footprint foot:PAD4 -> foot:PAD-4
- P10, P6, P7, P8, P9: footprint foot:PAD1 -> foot:PAD-1
- P11, P3, P4: footprint foot:PAD6 -> foot:PAD-6
- P5: footprint foot:PAD2 -> foot:PAD-2
- R36, R37: footprint foot:LR2512 -> foot:LR2512-D
- U1, U2, U3, U4: footprint foot:MSOP8 -> foot:MSOP-8
- Z1: footprint foot:SMD_Z3225 -> foot:SM-Z3225
